File: EP91Starlet.kicad_pcb (KiCad board)
At the start: 4 copper layers, 100 x 100 mm, 39 parts, among them M1 Module-vr-max9924-0.1, M2 Module-mega-mcu144-0.7, M3 Module-knock-0.2, M4 Module-wbo-0.5, M5 Module-vr-max9924-0.1, M6 Module-power_12and5V-0.3, Q1 ISL9V3040D3ST, Q2 ISL9V3040D3ST, Q3 ISL9V3040D3ST, Q4 ISL9V3040D3ST, U2 VNLD5160TR-E, U3 VNLD5160TR-E, U4 VNLD5160TR-E, U5 VNLD5160TR-E

Commit message: progress
Parts:
- F1, F2, F3, F4, R10, R11, R12, R13, R14, R15, R16, R9: moved to B.Cu
- moved M1 113.4 mm to (158.4, 57.4)
- moved M5 113.4 mm to (162.2, 72.8)
- moved M3 112.5 mm to (144.9, 137.5)
- moved M2 110.5 mm to (172.1, 129.6)
- moved M6 83.3 mm to (113.4, 62.1)
- moved M4 75.9 mm to (106.7, 99.8)
- moved F1 58.8 mm to (185.4, 93.2), turned to -90 degrees
- moved R9 53.2 mm to (186.9, 93.3), turned to 90 degrees
- moved R15 50.1 mm to (192.1, 112.7), turned to 0 degrees
- moved R16 49.9 mm to (192.1, 122.7), turned to 0 degrees
- moved R11 49.3 mm to (192.1, 92.7), turned to 0 degrees
- moved R12 49.1 mm to (192.1, 102.7), turned to 0 degrees
- moved Q4 38.3 mm to (194.6, 122.8)
- moved Q3 38.2 mm to (194.6, 112.8)
- moved Q2 37.2 mm to (194.6, 102.8)
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Routing:
- net Net-(M6-IN_VIGN): track 0.00 -> 100.8 mm

Commit message: inj wiring
Parts:
- moved R4 174.0 mm to (69.8, 107.7)
- moved R1 173.7 mm to (69.8, 101.9)
- moved R2 173.7 mm to (69.8, 110.2)
- moved R3 173.7 mm to (69.8, 99.3)
- moved D1 173.6 mm to (59.8, 105.8)
- moved D2 173.6 mm to (59.8, 109.3)
- moved D3 173.6 mm to (60.0, 97.7)
- moved D4 173.6 mm to (60.0, 101.2)
- moved R5 173.6 mm to (46.1, 99.9)
- moved R6 173.6 mm to (46.1, 108.3)
- moved R7 173.6 mm to (46.1, 97.4)
- moved U2 173.6 mm to (75.4, 101.2)
- moved U3 173.6 mm to (75.4, 109.6)
- moved U4 173.6 mm to (51.8, 107.4)
- moved U5 173.6 mm to (51.9, 99.3)
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Routing:
- net /IGN4/IN4: track 0.00 -> 23.2 mm
- net /IGN4/IN1: track 0.00 -> 18.7 mm
- net /IGN4/IN3: track 0.00 -> 16.4 mm
- net /IGN4/IN2: track 0.00 -> 15.0 mm
- net Net-(F4-Pad1): track 0.00 -> 3.34 mm
- net Net-(F3-Pad1): track 0.00 -> 3.34 mm
- net Net-(F2-Pad1): track 0.00 -> 3.34 mm
- net Net-(F1-Pad1): track 0.00 -> 3.34 mm

Commit message: start pcb routing
Parts:
- added J1: Conn_02x04_Top_Bottom, Connector_Molex:Molex_Mini-Fit_Jr_5569-08A2_2x04_P4.20mm_Horizontal, F.Cu at (180.8, 52.8)
- R1, R2, R3, R4, U2, U3: moved to B.Cu
- moved R3 93.2 mm to (159.8, 74.8), turned to 90 degrees
- moved R1 91.5 mm to (157.2, 74.8), turned to 90 degrees
- moved U2 88.5 mm to (157.9, 69.1), turned to 90 degrees
- moved R4 87.9 mm to (151.4, 74.8), turned to 90 degrees
- moved R2 86.6 mm to (148.8, 74.8), turned to 90 degrees
- moved U3 84.4 mm to (149.5, 69.3), turned to 90 degrees
- moved M3 72.9 mm to (136.0, 65.2), turned to -90 degrees
- moved D1 61.7 mm to (120.8, 96.5)
- moved D2 61.7 mm to (120.8, 100.1)
- moved R5 61.7 mm to (107.2, 90.7)
- moved R6 61.7 mm to (107.2, 99.1)
- moved R7 61.7 mm to (107.2, 88.1)
- moved R8 61.7 mm to (107.2, 96.3)
- moved U5 61.7 mm to (113.0, 90.0)
- moved D3 61.7 mm to (121.0, 88.4)
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Connections:
- M1 pad E4: +5VP -> +5VA
- M2 pad E38: unconnected-(M2-V5A_SWITCHABLE-PadE38) -> +5VA
- M2 pad W1: unconnected-(M2-GNDA-PadW1) -> GNDA
- M2 pad W2: unconnected-(M2-V5A_SWITCHABLE-PadW2) -> +5VA
- M4 pad J1: unconnected-(M4-SEL1-PadJ1) -> Net-(M4-PULL_DOWN1)
- M4 pad J_GND1: unconnected-(M4-PULL_DOWN1-PadJ_GND1) -> Net-(M4-PULL_DOWN1)
- M5 pad E4: +5VP -> +5VA
- U1 pad 2: /INJ4/OUT1 -> /INJ4/OUT4
- U1 pad 35: /IGN4/OUT1 -> /IGN4/OUT4
- U1 pad 41: /INJ4/OUT2 -> /INJ4/OUT3
Routing:
- net +5V: track 0.00 -> 94.1 mm
- net /INJ4/OUT3: track 0.00 -> 93.9 mm, vias 0 -> 1
- net /INJ4/OUT4: track 0.00 -> 84.8 mm, vias 0 -> 1
- net /CAN+: track 0.00 -> 83.7 mm
- net Net-(M2-VBAT): track 0.00 -> 82.0 mm
- net /CAN-: track 0.00 -> 81.2 mm
- net Net-(M2-IN_VIGN): track 0.00 -> 79.5 mm
- net /IGN4/OUT4: track 0.00 -> 67.3 mm
- net /INJ4/IN1: track 0.00 -> 63.3 mm, vias 0 -> 1
- net /INJ4/IN2: track 0.00 -> 62.1 mm, vias 0 -> 1
- net /INJ4/IN3: track 0.00 -> 49.0 mm
- net /INJ4/OUT1: track 0.00 -> 44.9 mm
- net /INJ4/OUT2: track 0.00 -> 42.9 mm
- net /INJ4/IN4: track 0.00 -> 42.1 mm
- net Net-(M6-IN_VIGN): track 100.8 -> 60.6 mm
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
Commit message: JLC test
Parts:
- M1, M5: footprint vrmax:vr-max9924 -> vrmax9924:vr-max9924
- M2: footprint mega_mcu144:mega-mcu144 -> megamcu144:mega-mcu144
- moved M5 3.54 mm to (192.3, 95.2)
- moved D4 1.99 mm to (119.5, 90.7)
- moved D2 1.80 mm to (119.5, 98.8)
- moved D3 1.55 mm to (119.5, 88.1)
- moved D1 1.30 mm to (119.5, 96.3)
Connections:
- M6 pad V1: Net-(M6-IN_VIGN) -> +12V_RAW
- M6 pad V2: Net-(M6-IN_VIGN) -> +12V_RAW
- M6 pad V3: Net-(M6-IN_VIGN) -> +12V_RAW
- U1 pad 23: Net-(M6-IN_VIGN) -> +12V_RAW
Routing:
- net +12V_RAW: track 0.00 -> 123.9 mm, vias 0 -> 4
- net Net-(M5-VR+): track 0.00 -> 112.9 mm
- net Net-(M1-VR+): track 0.00 -> 93.9 mm
- net Net-(M6-IN_VIGN): track 60.6 -> 0.00 mm
- net /IGN4/IN1: track 0.00 -> 55.8 mm
- net /IGN4/IN2: track 0.00 -> 45.5 mm
- net /IGN4/IN3: track 0.00 -> 35.8 mm
- net /IGN4/IN4: track 0.00 -> 35.0 mm
- net /LS_PROTECTED_2/OUT2: track 0.00 -> 4.96 mm
- net /FAN: track 0.00 -> 2.54 mm
- net /LS_PROTECTED_2/OUT1: track 0.00 -> 2.42 mm

Commit message: pcb layouting
Parts:
- added J2: Conn_02x03_Top_Bottom, Connector_Molex:Molex_Mini-Fit_Jr_5569-06A2_2x03_P4.20mm_Horizontal, F.Cu at (239.5, 93.3)
- R1, R2, R3, R4, U2, U3: moved to F.Cu
- moved R5 91.7 mm to (198.3, 99.9)
- moved R6 91.2 mm to (198.3, 101.9)
- moved U4 82.7 mm to (195.5, 95.7)
- moved R7 81.3 mm to (187.6, 99.9)
- moved M3 81.2 mm to (170.9, 138.5), turned to 0 degrees
- moved R8 80.7 mm to (187.6, 101.9)
- moved M4 79.6 mm to (170.3, 73.4), turned to 0 degrees
- moved D2 74.7 mm to (194.1, 103.6), turned to 0 degrees
- moved D1 74.7 mm to (194.1, 100.5), turned to 0 degrees
- moved U5 72.0 mm to (184.8, 95.7)
- moved D4 65.2 mm to (183.4, 103.6), turned to 0 degrees
- moved D3 65.1 mm to (183.4, 100.5), turned to 0 degrees
- moved Q4 62.7 mm to (230.5, 53.6), turned to 0 degrees
- moved R16 60.6 mm to (227.5, 53.6), turned to 0 degrees
- moved R14 57.9 mm to (223.0, 53.6), turned to -90 degrees
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Connections:
- M4 pad E1: unconnected-(M4-LSU_Un-PadE1) -> Net-(J2-Pin_4)
- M4 pad E2: unconnected-(M4-LSU_Vm-PadE2) -> Net-(J2-Pin_6)
- M4 pad E3: unconnected-(M4-LSU_Ip-PadE3) -> Net-(J2-Pin_3)
- M4 pad E4: unconnected-(M4-LSU_Rtrim-PadE4) -> Net-(J2-Pin_1)
- M4 pad E5: unconnected-(M4-LSU_H+-PadE5) -> Net-(J2-Pin_2)
Routing:
- net +12V_RAW: track 123.9 -> 0.00 mm, vias 4 -> 0
- net Net-(M5-VR+): track 112.9 -> 0.00 mm
- net +5V: track 94.1 -> 0.00 mm
- net /INJ4/OUT3: track 93.9 -> 0.00 mm, vias 1 -> 0
- net Net-(M1-VR+): track 93.9 -> 0.00 mm
- net /INJ4/OUT4: track 84.8 -> 0.00 mm, vias 1 -> 0
- net /CAN+: track 83.7 -> 0.00 mm
- net Net-(M2-VBAT): track 82.0 -> 0.00 mm
- net /CAN-: track 81.2 -> 0.00 mm
- net Net-(M2-IN_VIGN): track 79.5 -> 0.00 mm
- net /IGN4/OUT4: track 67.3 -> 0.00 mm
- net /INJ4/IN1: track 63.3 -> 0.00 mm, vias 1 -> 0
- net /INJ4/IN2: track 62.1 -> 0.00 mm, vias 1 -> 0
- net /IGN4/IN1: track 55.8 -> 0.00 mm
- net /INJ4/IN3: track 49.0 -> 0.00 mm
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
Commit message: jlc test
Parts:
- D1, D2, D3, D4, R5, R6, R7, R8, U4, U5: moved to B.Cu
- moved J2 133.5 mm to (111.3, 56.3), turned to 90 degrees
- moved Q1 88.9 mm to (154.8, 70.3), turned to 90 degrees
- moved R11 88.0 mm to (154.8, 73.3), turned to 90 degrees
- moved R9 87.1 mm to (154.8, 77.8), turned to 0 degrees
- moved F1 86.9 mm to (154.8, 79.3), turned to 180 degrees
- moved M1 76.7 mm to (103.1, 98.1), turned to -90 degrees
- moved Q2 75.2 mm to (164.8, 70.3), turned to 90 degrees
- moved R12 74.2 mm to (164.8, 73.3), turned to 90 degrees
- moved R10 73.1 mm to (164.8, 77.8), turned to 0 degrees
- moved F2 72.8 mm to (164.8, 79.3), turned to 180 degrees
- moved M5 70.2 mm to (103.1, 115.9), turned to -90 degrees
- moved Q3 61.7 mm to (174.8, 70.3), turned to 90 degrees
- moved R15 60.5 mm to (174.8, 73.3), turned to 90 degrees
- moved R13 59.1 mm to (174.8, 77.8), turned to 0 degrees
- moved F3 58.8 mm to (174.8, 79.3), turned to 180 degrees
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Connections:
- net /FAN renamed /RAD FAN
- D2 pad 2: /LS_PROTECTED_2/OUT2 -> /FUEL PUMP RELAY
- D3 pad 2: /LS_PROTECTED_2/OUT1 -> /CARBON CAN SOLENOID
- D4 pad 2: /LS_PROTECTED_2/OUT2 -> /IDLE UP SOLENOID
- F1 pad 2: /IGN4/IN1 -> /IGN4/IN4
- F2 pad 2: /IGN4/IN2 -> /IGN4/IN3
- F3 pad 2: /IGN4/IN3 -> /IGN4/IN2
- F4 pad 2: /IGN4/IN4 -> /IGN4/IN1
- M2 pad E31: /LS_PROTECTED_2/IN1 -> /LS_PROTECTED_2 A/IN1
- M2 pad E32: /LS_PROTECTED_2/IN2 -> /LS_PROTECTED_2 A/IN2
- M2 pad E33: /LS_PROTECTED_2/IN1 -> /LS_PROTECTED_2 B/IN1
- M2 pad E34: /LS_PROTECTED_2/IN2 -> /LS_PROTECTED_2 B/IN2
- M2 pad S13: unconnected-(M2-IN_AUX1-PadS13) -> /NEUTRAL STARTER SWITCH
- Q1 pad 2: /IGN4/OUT1 -> /IGN4/OUT4
- Q2 pad 2: /IGN4/OUT2 -> /IGN4/OUT3
- Q3 pad 2: /IGN4/OUT3 -> /IGN4/OUT2
- Q4 pad 2: /IGN4/OUT4 -> /IGN4/OUT1
- R1 pad 2: /INJ4/IN2 -> /INJ4/IN1
- R11 pad 2: /IGN4/OUT1 -> /IGN4/OUT4
- R12 pad 2: /IGN4/OUT2 -> /IGN4/OUT3
- R15 pad 2: /IGN4/OUT3 -> /IGN4/OUT2
- R16 pad 2: /IGN4/OUT4 -> /IGN4/OUT1
- R3 pad 2: /INJ4/IN1 -> /INJ4/IN2
- R5 pad 2: /LS_PROTECTED_2/IN2 -> /LS_PROTECTED_2 A/IN1
- R6 pad 2: /LS_PROTECTED_2/IN1 -> /LS_PROTECTED_2 A/IN2
- R7 pad 2: /LS_PROTECTED_2/IN2 -> /LS_PROTECTED_2 B/IN1
- R8 pad 2: /LS_PROTECTED_2/IN1 -> /LS_PROTECTED_2 B/IN2
- U1 pad 2: /INJ4/OUT4 -> /INJ4/OUT1
- U1 pad 24: unconnected-(U1-CCO-Pad24) -> /CARBON CAN SOLENOID
- U1 pad 25: unconnected-(U1-FC-Pad25) -> /FUEL PUMP RELAY
- U1 pad 31: unconnected-(U1-NSW-Pad31) -> /NEUTRAL STARTER SWITCH
- U1 pad 4: unconnected-(U1-IPV-Pad4) -> /IDLE UP SOLENOID
- U1 pad 9: unconnected-(U1-VCC-Pad9) -> +5VP
- U2 pad 1: /INJ4/IN1 -> /INJ4/IN2
- U2 pad 3: /INJ4/IN2 -> /INJ4/IN1
- U4 pad 1: /LS_PROTECTED_2/IN1 -> /LS_PROTECTED_2 A/IN2
- U4 pad 3: /LS_PROTECTED_2/IN2 -> /LS_PROTECTED_2 A/IN1
- U4 pad 6: /LS_PROTECTED_2/OUT2 -> /FUEL PUMP RELAY
- U5 pad 1: /LS_PROTECTED_2/IN1 -> /LS_PROTECTED_2 B/IN2
- U5 pad 3: /LS_PROTECTED_2/IN2 -> /LS_PROTECTED_2 B/IN1
- U5 pad 6: /LS_PROTECTED_2/OUT2 -> /IDLE UP SOLENOID
- U5 pad 8: /LS_PROTECTED_2/OUT1 -> /CARBON CAN SOLENOID
Routing:
- net /INJ4/OUT1: track 0.00 -> 139.2 mm, vias 0 -> 5
- net /INJ4/OUT3: track 0.00 -> 134.8 mm, vias 0 -> 3
- net /IGN4/OUT4: track 0.00 -> 85.9 mm, vias 0 -> 6
- net /IGN4/IN1: track 0.00 -> 82.0 mm, vias 0 -> 1
- net /INJ4/OUT2: track 0.00 -> 77.4 mm, vias 0 -> 3
- net /IGN4/IN2: track 0.00 -> 73.5 mm, vias 0 -> 1
- net /IGN4/IN3: track 0.00 -> 65.6 mm, vias 0 -> 1
- net /INJ4/IN3: track 0.00 -> 58.6 mm, vias 0 -> 2
- net /INJ4/IN2: track 0.00 -> 57.7 mm, vias 0 -> 2
- net /INJ4/IN4: track 0.00 -> 57.7 mm, vias 0 -> 2
- net /IGN4/IN4: track 0.00 -> 57.5 mm, vias 0 -> 1
- net /INJ4/OUT4: track 0.00 -> 57.0 mm, vias 0 -> 1
- net /INJ4/IN1: track 0.00 -> 55.4 mm, vias 0 -> 2
- net +12V_RAW: track 0.00 -> 54.3 mm
- net /IGN4/OUT3: track 0.00 -> 35.3 mm, vias 0 -> 2
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