File: EP91Starlet.kicad_pcb (KiCad board)
At the start: 4 copper layers, 100 x 100 mm, 71 parts, among them J1 175446-6, J2 USB_B, J3 Conn_01x02, J5 Conn_01x02, J6 Conn_02x03_Top_Bottom, J7 Conn_02x20_Odd_Even, J9 Conn_02x06_Top_Bottom, M1 Module-mega-mcu144-0.7, M2 Module-vr-max9924-0.1, M3 Module-vr-discrete-0.5, M4 Module-power_12and5V-0.3, M5 Module-wbo-0.6, M6 Module-knock-0.2, M7 Module-can-0.1, Q2 BSS138, U1 VNLD5090-E, U2 VNLD5090-E, U3 VNLD5090-E, U4 VNLD5090-E, U5 VNLD5090-E, U6 VNLD5090-E, U7 MAX31855KASA, U8 TLE9201SG

Commit message: sync
Parts:
- removed J2: USB_B, kicad6-libraries:USB_B
- added J4: USB_B_Mini, Connector_USB:USB_Mini-B_Wuerth_65100516121_Horizontal, F.Cu at (211.0, 117.2)
- moved C12 81.2 mm to (158.7, 133.9)
- moved C15 81.2 mm to (158.7, 141.4)
- moved C11 81.2 mm to (158.7, 131.4)
- moved C13 81.2 mm to (158.7, 136.4)
- moved C14 81.2 mm to (158.7, 138.9)
- moved C10 81.2 mm to (154.7, 141.4)
- moved C7 81.2 mm to (154.7, 133.9)
- moved C8 81.2 mm to (154.7, 136.4)
- moved C9 81.2 mm to (154.7, 138.9)
- moved C6 79.9 mm to (155.8, 130.6)
- moved C16 76.2 mm to (168.7, 132.6), turned to -90 degrees
- moved R15 67.2 mm to (184.1, 148.8)
- moved C17 65.2 mm to (189.5, 147.4)
- moved C18 65.2 mm to (189.5, 149.9)
- moved J9 50.2 mm to (214.1, 141.6), turned to 180 degrees
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Connections:
- J9 pad 11: /LS3_OUT -> /DC1+
- J9 pad 12: /LS4_OUT -> /DC1-
- J9 pad 7: /DC1+ -> /LS3_OUT
- J9 pad 8: /DC1- -> /LS4_OUT
