File: EP91Starlet.kicad_pcb (KiCad board)
At the start: 4 copper layers, 100 x 100 mm, 71 parts, among them J1 175446-6, J3 Conn_01x02, J4 USB_B_Mini, J5 Conn_01x02, J6 Conn_02x03_Top_Bottom, J7 Conn_02x20_Odd_Even, J9 Conn_02x06_Top_Bottom, M1 Module-mega-mcu144-0.7, M2 Module-vr-max9924-0.1, M3 Module-vr-discrete-0.5, M4 Module-power_12and5V-0.3, M5 Module-wbo-0.6, M6 Module-knock-0.2, M7 Module-can-0.1, Q2 BSS138, U1 VNLD5090-E, U2 VNLD5090-E, U3 VNLD5090-E, U4 VNLD5090-E, U5 VNLD5090-E, U6 VNLD5090-E, U7 MAX31855KASA, U8 TLE9201SG

Commit message: sync
Parts:
- removed TP1: TestPoint, TestPoint:TestPoint_Pad_D1.0mm
- removed U1, U2, U3, U4, U5, U6: VNLD5090-E, VNLD5090-E:VNLD5090-E
- added IC1: VNLD5160-E, VNLD5160-E:SOIC127P600X175-8N, F.Cu at (219.4, 53.9)
- added IC2: VNLD5160-E, VNLD5160-E:SOIC127P600X175-8N, F.Cu at (232.7, 54.9)
- added IC3: VNLD5160-E, VNLD5160-E:SOIC127P600X175-8N, B.Cu at (153.5, 34.5)
- added IC4: VNLD5160-E, VNLD5160-E:SOIC127P600X175-8N, B.Cu at (134.5, 33.8)
- added IC5: VNLD5160-E, VNLD5160-E:SOIC127P600X175-8N, F.Cu at (223.8, 81.0)
- added IC6: VNLD5160-E, VNLD5160-E:SOIC127P600X175-8N, F.Cu at (232.7, 81.1)
- added REF**: MountingHole_3.2mm_M3_Pad_Via, MountingHole:MountingHole_3.2mm_M3_Pad_Via, F.Cu at (207.1, 33.9)
- added REF**1: MountingHole_3.2mm_M3_Pad_Via, MountingHole:MountingHole_3.2mm_M3_Pad_Via, F.Cu at (114.3, 33.9)
- added REF**2: MountingHole_3.2mm_M3_Pad_Via, MountingHole:MountingHole_3.2mm_M3_Pad_Via, F.Cu at (207.1, 126.7)
- added REF**3: MountingHole_3.2mm_M3_Pad_Via, MountingHole:MountingHole_3.2mm_M3_Pad_Via, F.Cu at (114.3, 126.7)
- BT1: moved to F.Cu
- D1, D2, D3, D4, R5, R6, R7, R8: moved to B.Cu
- J1: footprint TE-175446-6:1754466 -> TE_175446-6:1754466
- J6: footprint New_Connector_Molex:Molex_Mini-Fit_Jr_5566-06A_2x03_P4.20mm_Vertical -> Connector_Molex:Molex_Mini-Fit_Jr_5566-06A_2x03_P4.20mm_Vertical
- J9: footprint New_Connector_Molex:Molex_Mini-Fit_Jr_5566-12A_2x06_P4.20mm_Vertical -> Connector_Molex:Molex_Mini-Fit_Jr_5566-12A_2x06_P4.20mm_Vertical
- M4: footprint hellen-one-power_12and5V:power_12and5V -> hellen-one-power_12and5V-0.3:power_12and5V
- moved F1 213.1 mm to (28.3, 96.4)
- moved C17 156.7 mm to (73.8, 41.7)
- moved C18 156.7 mm to (73.8, 44.2)
- moved C1 152.4 mm to (102.6, 45.0)
- moved C2 152.4 mm to (102.6, 47.5)
- moved C3 152.4 mm to (102.6, 50.0)
- moved C4 152.4 mm to (102.6, 52.5)
- moved C5 152.4 mm to (102.6, 55.0)
- moved R15 150.3 mm to (73.8, 46.7)
- moved U8 145.9 mm to (77.0, 33.8)
- moved D10 140.1 mm to (96.2, 54.5)
- moved C16 133.2 mm to (73.8, 39.2), turned to 0 degrees
- moved L1 128.6 mm to (102.6, 57.5)
- moved L2 128.6 mm to (102.6, 60.1)
- moved C6 128.3 mm to (65.8, 39.2)
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Connections:
- net Net-(J4-VBUS) renamed /USB+
- D1 pad 2: /FANRELAY_OUT -> /FUELRELAY_OUT
- D4 pad 2: /IACOPEN_OUT -> /IACCLOSE_OUT
- D7 pad 2: /LS2_OUT -> /LS1_OUT
- D9 pad 2: /LS4_OUT -> /LS3_OUT
- J7 pad 18: /CAN1- -> /CAN1+
- J7 pad 20: /CAN1+ -> /CAN1-
- J9 pad 1: +12V_RAW -> GND
- M1 pad W12: /CAN2+ -> /CAN1+
- M1 pad W13: /CAN2- -> /CAN1-
- M7 pad S1: /CAN1- -> /CAN2+
- M7 pad S2: /CAN1+ -> /CAN2-
- R5 pad 1: /FUELRELAY_IN -> /FANRELAY_IN
- R6 pad 1: /FANRELAY_IN -> /FUELRELAY_IN
Routing:
- net /THRESH: track 72.7 -> 0.00 mm
- net Net-(M1-SPI2_SCK/CAN2_TX): track 66.3 -> 0.00 mm
- net Net-(M1-SPI2_CS/CAN2_RX): track 63.2 -> 0.00 mm
- net /5V_OUT1: track 58.3 -> 0.00 mm
- net /VSS: track 55.7 -> 0.00 mm, vias 1 -> 0
- net /CAN2-: track 54.8 -> 0.00 mm
- net /5V_OUT2: track 53.7 -> 0.00 mm
- net /CAN2+: track 52.3 -> 0.00 mm
- net /5V_OUT3: track 49.2 -> 0.00 mm
- net /5V_OUT4: track 44.6 -> 0.00 mm
- net /5V_OUT5: track 40.0 -> 0.00 mm
- net +5V: track 41.5 -> 80.5 mm
- net /SPARK: track 37.2 -> 0.00 mm
- net +5VA: track 32.2 -> 0.00 mm
- net +12V_PERM: track 75.7 -> 97.6 mm
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Other:
- outline, holes or cut-outs redrawn
