File: EP91Starlet.kicad_sch (KiCad schematic)
At the start: 7 parts, among them M1 Module-vr-max9924-0.1, M2 Module-mega-mcu144-0.7, M3 Module-knock-0.2, M4 Module-wbo-0.5, M5 Module-vr-max9924-0.1, M6 Module-power_12and5V-0.3

Commit message: start pcb routing
Parts:
- added J1: Conn_02x04_Top_Bottom, Connector_Molex:Molex_Mini-Fit_Jr_5569-08A2_2x04_P4.20mm_Horizontal, symbol Connector_Generic:Conn_02x04_Top_Bottom
Connections:
- net LS_PROTECTED_2/IN1 is gone; now on net LS_PROTECTED_2/IN1: M2.E33 (OUT_INJ7)
- net LS_PROTECTED_2/IN2 is gone; now on net LS_PROTECTED_2/IN2: M2.E34 (OUT_INJ8)
- net +5VA: now also M1.E4 (V5_IN), M2.E38 (V5A_SWITCHABLE), M2.W2 (V5A_SWITCHABLE), M5.E4 (V5_IN)
- net +5VP: no longer M1.E4 (V5_IN), M5.E4 (V5_IN)
- net IGN4/OUT1: now also J1.8 (Pin_8); no longer U1.35 (IGT)
- net IGN4/OUT2: now also J1.7 (Pin_7)
- net IGN4/OUT3: now also J1.6 (Pin_6)
- net IGN4/OUT4: now also U1.35 (IGT), J1.5 (Pin_5)
- net INJ4/OUT1: now also J1.4 (Pin_4); no longer U1.2 (#20)
- net INJ4/OUT2: now also J1.3 (Pin_3); no longer U1.41 (#10)
- net INJ4/OUT3: now also U1.41 (#10), J1.2 (Pin_2)
- net INJ4/OUT4: now also U1.2 (#20), J1.1 (Pin_1)
- net LS_PROTECTED_2/IN1: no longer M2.E31 (OUT_INJ5)
- net LS_PROTECTED_2/IN2: no longer M2.E32 (OUT_INJ6)
- net GNDA: now reaches M2.W1 (GNDA)
- net at M4.J1 (SEL1): now also M4.J_GND1 (PULL_DOWN1)
- new net LS_PROTECTED_2/IN1: M2.E31 (OUT_INJ5)
- new net LS_PROTECTED_2/IN2: M2.E32 (OUT_INJ6)
- no-connect marks 4 -> 9

Commit message: JLC test
Parts:
- M1, M5: footprint vrmax:vr-max9924 -> vrmax9924:vr-max9924
- M2: footprint mega_mcu144:mega-mcu144 -> megamcu144:mega-mcu144
Connections:
- net LS_PROTECTED_2/IN1 is gone; now on net LS_PROTECTED_2/IN1: M2.E33 (OUT_INJ7)
- net LS_PROTECTED_2/IN2 is gone; now on net LS_PROTECTED_2/IN2: M2.E34 (OUT_INJ8)
- net LS_PROTECTED_2/IN1: no longer M2.E31 (OUT_INJ5)
- net LS_PROTECTED_2/IN2: no longer M2.E32 (OUT_INJ6)
- net +12V_RAW: now reaches M6.V1 (V12_PERM), M6.V2 (IN_VIGN), M6.V3 (V12_RAW), U1.23 (BATT)
- new net LS_PROTECTED_2/IN1: M2.E31 (OUT_INJ5)
- new net LS_PROTECTED_2/IN2: M2.E32 (OUT_INJ6)
Changed lines of the file:
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@@
+	)
+	(junction
+		(at 86.36 195.58)
+		(diameter 0)
+		(color 0 0 0 0)
 	)
 	(junction
@@
 	(wire
 		(pts
-			(xy 88.9 195.58) (xy 76.2 195.58)
+			(xy 88.9 195.58) (xy 86.36 195.58)
 		)
 		(stroke
@@
 		(pts
 			(xy 99.06 25.4) (xy 99.06 36.83)
+		)
+		(stroke
+			(width 0)
+			(type default)
+		)
+	)
+	(wire
+		(pts
+			(xy 86.36 195.58) (xy 76.2 195.58)
 		)
 		(stroke
@@
 			)
 		)
-		(property "Footprint" "vrmax:vr-max9924"
+		(property "Footprint" "vrmax9924:vr-max9924"
 			(at 120.65 133.35 0)
 			(effects
@@
 			)
 		)
-		(property "Footprint" "mega_mcu144:mega-mcu144"
+		(property "Footprint" "megamcu144:mega-mcu144"
 			(at 175.26 25.4 0)
 			(effects
@@
 				(path "/10fbc709-889c-4565-8161-129ca9f0b73f"
 					(reference "M2")
+					(unit 1)
+				)
+			)
+		)
+	)
+	(symbol
+		(lib_id "misc:+12V_RAW")
+		(at 86.36 195.58 0)
+		(unit 1)
+		(exclude_from_sim no)
+		(in_bom yes)
+		(on_board yes)
+		(dnp no)
+		(fields_autoplaced yes)
+		(property "Reference" "#PWR38"
+			(at 86.36 199.39 0)
+			(effects
+				(font
+					(size 1.27 1.27)
+				)
+				(hide yes)
+			)
+		)
+		(property "Value" "+12V_RAW"
+			(at 86.36 190.5 0)
+			(effects
+				(font
+					(size 1.27 1.27)
+				)
+			)
+		)
+		(property "Footprint" ""
+			(at 86.36 195.58 0)
+			(effects
+				(font
+					(size 1.27 1.27)
+				)
+				(hide yes)
+			)
+		)
+		(property "Datasheet" ""
+			(at 86.36 195.58 0)
+			(effects
+				(font
+					(size 1.27 1.27)
+				)
+				(hide yes)
+			)
+		)
+		(property "Description" "Power symbol creates a global label with name \"+12V_RAW\""
+			(at 86.36 195.58 0)
+			(effects
+				(font
+					(size 1.27 1.27)
+				)
+				(hide yes)
+			)
+		)
+		(pin "1"
+		)
+		(instances
+			(project ""
+				(path "/10fbc709-889c-4565-8161-129ca9f0b73f"
+					(reference "#PWR38")
 					(unit 1)
 				)
@@
 			)
 		)
-		(property "Footprint" "vrmax:vr-max9924"
+		(property "Footprint" "vrmax9924:vr-max9924"
 			(at 120.65 156.21 0)
 			(effects

Commit message: pcb layouting
Parts:
- added J2: Conn_02x03_Top_Bottom, Connector_Molex:Molex_Mini-Fit_Jr_5569-06A2_2x03_P4.20mm_Horizontal, symbol Connector_Generic:Conn_02x03_Top_Bottom
Connections:
- net LS_PROTECTED_2/IN1 is gone; now on net LS_PROTECTED_2/IN1: M2.E33 (OUT_INJ7)
- net LS_PROTECTED_2/IN2 is gone; now on net LS_PROTECTED_2/IN2: M2.E34 (OUT_INJ8)
- net +12V_RAW: now also J2.5 (Pin_5)
- net +5VP: now also U1.9 (VCC)
- net INJ4/OUT2: now also U1.41 (#10)
- net INJ4/OUT3: no longer U1.41 (#10)
- net LS_PROTECTED_2/IN1: no longer M2.E31 (OUT_INJ5)
- net LS_PROTECTED_2/IN2: no longer M2.E32 (OUT_INJ6)
- net CARBON CAN SOLENOID: now reaches U1.24 (CCO)
- net FUEL PUMP RELAY: now reaches U1.25 (FC)
- net NEUTRAL STARTER SWITCH: now reaches U1.31 (NSW)
- net NEUTRAL STARTER SWITCH: now also M2.S13 (IN_AUX1)
- net IDLE UP SOLENOID: now reaches U1.4 (IPV)
- net at M4.E1 (LSU_Un): now also J2.4 (Pin_4)
- net at M4.E2 (LSU_Vm): now also J2.6 (Pin_6)
- net at M4.E3 (LSU_Ip): now also J2.3 (Pin_3)
- net at M4.E4 (LSU_Rtrim): now also J2.1 (Pin_1)
- net at M4.E5 (LSU_H+): now also J2.2 (Pin_2)
- net FAN renamed RAD FAN
- new net LS_PROTECTED_2/IN1: M2.E31 (OUT_INJ5)
- new net LS_PROTECTED_2/IN2: M2.E32 (OUT_INJ6)
- no-connect marks 9 -> 18
Other:
- note added: "IDL: idle switch in tps to show if at 0 throttle HT: narrowband o2 sensor heater ~: ??? FAN: turns rad fan off or on (LS) ELS1: recieves input signal with headlights on? ELS2: monitors rear defogger or heater blower motor? ELS3: recieves input signal when a/c clutch engaged? RSO: rotary solenoid open RSC: rotary solenoid close - cold idle speed control TE1: diagnostic port TE2: diagnostic port VF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"
- note added: "chosen out 4 and out 2 as they are on different components, split the load of batch injection"

Commit message: jlc test
Connections:
- net INJ4/OUT1: now also U1.2 (#20)
- net INJ4/OUT2: no longer U1.41 (#10)
- net INJ4/OUT3: now also U1.41 (#10)
- net INJ4/OUT4: no longer U1.2 (#20)
- net LS_PROTECTED_2 A/IN1 renamed LS_PROTECTED_2 B/IN1
- net LS_PROTECTED_2 A/IN2 renamed LS_PROTECTED_2 B/IN2
Other:
- sheet LS_PROTECTED_2 renamed LS_PROTECTED_2 A
- added sheet LS_PROTECTED_2 B (LSPROT2.kicad_sch)
