File: EP91Starlet.kicad_sch (KiCad schematic)
At the start: 46 parts, among them J1 175446-6, J2 USB_B, J3 Conn_01x02, J5 Conn_01x02, J6 Conn_02x03_Top_Bottom, J7 Conn_02x20_Odd_Even, J9 Conn_02x06_Top_Bottom, M1 Module-mega-mcu144-0.7, M2 Module-vr-max9924-0.1, M3 Module-vr-discrete-0.5, M4 Module-power_12and5V-0.3, M5 Module-wbo-0.6, M6 Module-knock-0.2, M7 Module-can-0.1, Q2 BSS138, U1 VNLD5090-E, U2 VNLD5090-E, U3 VNLD5090-E, U4 VNLD5090-E, U5 VNLD5090-E, U6 VNLD5090-E

Commit message: sync
Parts:
- removed J2: USB_B, kicad6-libraries:USB_B, symbol misc:USB_B
- added J4: USB_B_Mini, Connector_USB:USB_Mini-B_Wuerth_65100516121_Horizontal, symbol Connector:USB_B_Mini
Connections:
- net DC1+: now also J9.11 (Pin_11); no longer J9.7 (Pin_7)
- net DC1-: now also J9.12 (Pin_12); no longer J9.8 (Pin_8)
- net GND: now also J4.5 (GND), J4.6 (Shield)
- net LS3_OUT: now also J9.7 (Pin_7); no longer J9.11 (Pin_11)
- net LS4_OUT: now also J9.8 (Pin_8); no longer J9.12 (Pin_12)
- net at M1.N2 (USBM): now also J4.2 (D-)
- net at M1.N3 (USBP): now also J4.3 (D+)
- net at M1.N4 (VBUS): now also J4.1 (VBUS)
- no-connect marks 30 -> 31
Changed lines of the file:
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@@
 	)
 	(junction
-		(at 270.51 106.68)
-		(diameter 0)
-		(color 0 0 0 0)
-	)
-	(junction
 		(at 30.48 31.75)
 		(diameter 0)
@@
 	)
 	(junction
+		(at 270.51 106.68)
+		(diameter 0)
+		(color 0 0 0 0)
+	)
+	(junction
 		(at 69.85 226.06)
 		(diameter 0)
@@
 	)
 	(no_connect
+		(at 262.89 101.6)
+	)
+	(no_connect
 		(at 71.12 104.14)
 	)
@@
 		)
 	)
+	(label "DC1-"
+		(at 332.74 120.65 0)
+		(effects
+			(font
+				(size 1.27 1.27)
+			)
+			(justify left bottom)
+		)
+	)
 	(label "AUX4"
 		(at 369.57 113.03 180)
@@
 		)
 	)
+	(label "DC1+"
+		(at 332.74 118.11 0)
+		(effects
+			(font
+				(size 1.27 1.27)
+			)
+			(justify left bottom)
+		)
+	)
 	(label "MAP2"
 		(at 369.57 130.81 180)
@@
 		)
 	)
+	(label "LS3_OUT"
+		(at 332.74 107.95 0)
+		(effects
+			(font
+				(size 1.27 1.27)
+			)
+			(justify left bottom)
+		)
+	)
 	(label "LS2_HOT_IN"
 		(at 190.5 48.26 180)
@@
 		)
 	)
+	(label "LS4_OUT"
+		(at 332.74 110.49 0)
+		(effects
+			(font
+				(size 1.27 1.27)
+			)
+			(justify left bottom)
+		)
+	)
 	(label "PWR_EN"
 		(at 190.5 248.92 180)
@@
 		)
 	)
-	(label "LS3_OUT"
-		(at 332.74 118.11 0)
-		(effects
-			(font
-				(size 1.27 1.27)
-			)
-			(justify left bottom)
-		)
-	)
 	(label "VIGN"
 		(at 78.74 328.93 0)
@@
 		)
 	)
-	(label "DC1+"
-		(at 332.74 107.95 0)
-		(effects
-			(font
-				(size 1.27 1.27)
-			)
-			(justify left bottom)
-		)
-	)
 	(label "SENS1"
 		(at 369.57 110.49 180)
@@
 		)
 	)
-	(label "LS4_OUT"
-		(at 332.74 120.65 0)
-		(effects
-			(font
-				(size 1.27 1.27)
-			)
-			(justify left bottom)
-		)
-	)
 	(label "VR-"
 		(at 30.48 281.94 180)
@@
 		)
 	)
-	(label "DC1-"
-		(at 332.74 110.49 0)
-		(effects
-			(font
-				(size 1.27 1.27)
-			)
-			(justify left bottom)
-		)
-	)
 	(label "AIR"
 		(at 346.71 238.76 180)
@@
 	)
 	(symbol
+		(lib_id "Connector:USB_B_Mini")
+		(at 270.51 96.52 0)
+		(mirror y)
+		(unit 1)
+		(exclude_from_sim no)
+		(in_bom yes)
+		(on_board yes)
+		(dnp no)
+		(fields_autoplaced yes)
+		(property "Reference" "J4"
+			(at 276.86 95.2499 0)
+			(effects
+				(font
+					(size 1.27 1.27)
+				)
+				(justify right)
+			)
+		)
+		(property "Value" "USB_B_Mini"
+			(at 276.86 97.7899 0)
+			(effects
+				(font
+					(size 1.27 1.27)
+				)
+				(justify right)
+			)
+		)
+		(property "Footprint" "Connector_USB:USB_Mini-B_Wuerth_65100516121_Horizontal"
+			(at 266.7 97.79 0)
+			(effects
+				(font
+					(size 1.27 1.27)
+				)
+				(hide yes)
+			)
+		)
+		(property "Datasheet" "~"
+			(at 266.7 97.79 0)
+			(effects
+				(font
+					(size 1.27 1.27)
+				)
+				(hide yes)
+			)
+		)
+		(property "Description" "USB Mini Type B connector"
+			(at 270.51 96.52 0)
+			(effects
+				(font
+					(size 1.27 1.27)
+				)
+				(hide yes)
+			)
+		)
+		(pin "4"
+		)
+		(pin "5"
+		)
+		(pin "6"
+		)
+		(pin "2"
+		)
+		(pin "3"
+		)
+		(pin "1"
+		)
+		(instances
+			(project ""
+				(path "/10fbc709-889c-4565-8161-129ca9f0b73f"
+					(reference "J4")
+					(unit 1)
+				)
+			)
+		)
+	)
+	(symbol
 		(lib_id "Device:D")
 		(at 33.02 135.89 270)
@@
 					(unit 1)
 				)
-			)
-		)
-	)
-	(symbol
-		(lib_id "misc:USB_B")
-		(at 270.51 96.52 0)
-		(mirror y)
-		(unit 1)
-		(exclude_from_sim no)
-		(in_bom yes)
-		(on_board yes)
-		(dnp no)
-		(property "Reference" "J2"
-			(at 276.86 97.7901 0)
-			(effects
-				(font
-					(size 1.27 1.27)
-				)
-				(justify right)
-			)
-		)
-		(property "Value" "USB_B"
-			(at 276.86 95.2501 0)
-			(effects
-				(font
-					(size 1.27 1.27)
-				)
-				(justify right)
-			)
-		)
-		(property "Footprint" "kicad6-libraries:USB_B"
-			(at 266.7 97.79 0)
-			(effects
-				(font
-					(size 1.27 1.27)
-				)
-				(hide yes)
-			)
-		)
-		(property "Datasheet" "~"
-			(at 266.7 97.79 0)
-			(effects
-				(font
-					(size 1.27 1.27)
-				)
-				(hide yes)
-			)
-		)
-		(property "Description" "USB Type B connector"
-			(at 270.51 96.52 0)
-			(effects
-				(font
-					(size 1.27 1.27)
-				)
-				(hide yes)
-			)
-		)
-		(property "LCSC" "C46392"
-			(at 270.51 96.52 0)
-			(effects
-				(font
-					(size 1.27 1.27)
-				)
-				(hide yes)
-			)
-		)
-		(pin "5"
-		)
-		(pin "4"
-		)
-		(pin "2"
-		)
-		(pin "3"
-		)
-		(pin "1"
-		)
-		(instances
-			(project ""
-				(path "/10fbc709-889c-4565-8161-129ca9f0b73f"
-					(reference "J2")
-					(unit 1)
-				)
