File: EP91Starlet.kicad_sch (KiCad schematic)
At the start: 46 parts, among them J1 175446-6, J3 Conn_01x02, J4 USB_B_Mini, J5 Conn_01x02, J6 Conn_02x03_Top_Bottom, J7 Conn_02x20_Odd_Even, J9 Conn_02x06_Top_Bottom, M1 Module-mega-mcu144-0.7, M2 Module-vr-max9924-0.1, M3 Module-vr-discrete-0.5, M4 Module-power_12and5V-0.3, M5 Module-wbo-0.6, M6 Module-knock-0.2, M7 Module-can-0.1, Q2 BSS138, U1 VNLD5090-E, U2 VNLD5090-E, U3 VNLD5090-E, U4 VNLD5090-E, U5 VNLD5090-E, U6 VNLD5090-E

Commit message: sync
Parts:
- removed U1, U2, U3, U4, U5, U6: VNLD5090-E, VNLD5090-E:VNLD5090-E, symbol VNLD5090-E:VNLD5090-E
- added IC1, IC2, IC3, IC4, IC5, IC6: VNLD5160-E, VNLD5160-E:SOIC127P600X175-8N, symbol VNLD5160-E:VNLD5160TR-E
- J1: footprint TE-175446-6:1754466 -> TE_175446-6:1754466
- J6: footprint New_Connector_Molex:Molex_Mini-Fit_Jr_5566-06A_2x03_P4.20mm_Vertical -> Connector_Molex:Molex_Mini-Fit_Jr_5566-06A_2x03_P4.20mm_Vertical
- J9: footprint New_Connector_Molex:Molex_Mini-Fit_Jr_5566-12A_2x06_P4.20mm_Vertical -> Connector_Molex:Molex_Mini-Fit_Jr_5566-12A_2x06_P4.20mm_Vertical
- M4: footprint hellen-one-power_12and5V:power_12and5V -> hellen-one-power_12and5V-0.3:power_12and5V
Connections:
- net +12V_RAW: no longer J9.1 (Pin_1)
- net CAN1+: now also J7.18 (Pin_18), M1.W12 (CANH); no longer J7.20 (Pin_20), M7.S2 (CANH)
- net CAN1-: now also J7.20 (Pin_20), M1.W13 (CANL); no longer J7.18 (Pin_18), M7.S1 (CANL)
- net CAN2+: now also M7.S1 (CANL); no longer M1.W12 (CANH)
- net CAN2-: now also M7.S2 (CANH); no longer M1.W13 (CANL)
- net FANRELAY_IN: now also R5.1, IC4.3 (IN2); no longer R6.1
- net FANRELAY_OUT: now also IC4.8 (DRAIN1); no longer D1.2 (A)
- net FUELRELAY_IN: now also R6.1, IC4.1 (IN1); no longer R5.1
- net FUELRELAY_OUT: now also D1.2 (A), IC4.6 (DRAIN2)
- net GND: now also J9.1 (Pin_1), IC1.5 (SOURCE2), IC1.7 (SOURCE1), IC2.5 (SOURCE2), IC2.7 (SOURCE1), IC3.5 (SOURCE2), IC3.7 (SOURCE1), IC4.5 (SOURCE2), IC4.7 (SOURCE1), IC5.5 (SOURCE2), IC5.7 (SOURCE1), IC6.5 (SOURCE2), IC6.7 (SOURCE1)
- net IACCLOSE_IN: now also IC3.1 (IN1)
- net IACCLOSE_OUT: now also D4.2 (A), IC3.8 (DRAIN1)
- net IACOPEN_IN: now also IC3.3 (IN2)
- net IACOPEN_OUT: now also IC3.6 (DRAIN2); no longer D4.2 (A)
- net LS1_HOT_IN: now also IC6.1 (IN1)
- net LS1_HOT_OUT: now also IC6.8 (DRAIN1)
- net LS1_IN: now also IC2.1 (IN1)
- net LS1_OUT: now also D7.2 (A), IC2.8 (DRAIN1)
- net LS2_HOT_IN: now also IC6.3 (IN2)
- net LS2_HOT_OUT: now also IC6.6 (DRAIN2)
- net LS2_IN: now also IC2.3 (IN2)
- net LS2_OUT: now also IC2.6 (DRAIN2); no longer D7.2 (A)
- net LS3_HOT_IN: now also IC5.1 (IN1)
- net LS3_HOT_OUT: now also IC5.8 (DRAIN1)
- net LS3_IN: now also IC1.1 (IN1)
- net LS3_OUT: now also D9.2 (A), IC1.8 (DRAIN1)
- net LS4_HOT_IN: now also IC5.3 (IN2)
- net LS4_HOT_OUT: now also IC5.6 (DRAIN2)
- net LS4_IN: now also IC1.3 (IN2)
- net LS4_OUT: now also IC1.6 (DRAIN2); no longer D9.2 (A)
- net USB+: now reaches J4.1 (VBUS), M1.N4 (VBUS)
- net USB+: now also J4.2 (D-), J4.3 (D+), M1.N2 (USBM), M1.N3 (USBP)
- no-connect marks 31 -> 33
