File: IGN4.kicad_sch (KiCad schematic)
At the start: 16 parts, among them Q1 ISL9V3040D3ST, Q2 ISL9V3040D3ST, Q3 ISL9V3040D3ST, Q4 ISL9V3040D3ST

Commit message: jlc test
Connections:
- net IN1: now also F4.2; no longer F1.2
- net IN2: now also F3.2; no longer F2.2
- net IN3: now also F2.2; no longer F3.2
- net IN4: now also F1.2; no longer F4.2
- net OUT1: now also Q4.2 (C), R16.2; no longer Q1.2 (C), R11.2
- net OUT2: now also Q3.2 (C), R15.2; no longer Q2.2 (C), R12.2
- net OUT3: now also Q2.2 (C), R12.2; no longer Q3.2 (C), R15.2
- net OUT4: now also Q1.2 (C), R11.2; no longer Q4.2 (C), R16.2
Changed lines of the file:
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@@
 		)
 	)
-	(hierarchical_label "OUT1"
+	(hierarchical_label "OUT4"
 		(shape output)
 		(at 120.65 72.39 180)
@@
 		)
 	)
-	(hierarchical_label "IN4"
+	(hierarchical_label "IN1"
 		(shape input)
 		(at 198.12 105.41 0)
@@
 		)
 	)
-	(hierarchical_label "OUT4"
+	(hierarchical_label "OUT1"
 		(shape output)
 		(at 167.64 100.33 180)
@@
 		)
 	)
-	(hierarchical_label "IN1"
+	(hierarchical_label "IN4"
 		(shape input)
 		(at 151.13 77.47 0)
@@
 		)
 	)
-	(hierarchical_label "IN2"
+	(hierarchical_label "IN3"
 		(shape input)
 		(at 151.13 105.41 0)
@@
 		)
 	)
-	(hierarchical_label "OUT2"
+	(hierarchical_label "OUT3"
 		(shape output)
 		(at 120.65 100.33 180)
@@
 		)
 	)
-	(hierarchical_label "OUT3"
+	(hierarchical_label "OUT2"
 		(shape output)
 		(at 167.64 72.39 180)
@@
 		)
 	)
-	(hierarchical_label "IN3"
+	(hierarchical_label "IN2"
 		(shape input)
 		(at 198.12 77.47 0)
