File: INJ4.kicad_sch (KiCad schematic)
At the start: 6 parts, among them U2 VNLD5160TR-E, U3 VNLD5160TR-E

Commit message: jlc test
Connections:
- net IN1: now also R1.2, U2.3 (IN2); no longer R3.2, U2.1 (IN1)
- net IN2: now also R3.2, U2.1 (IN1); no longer R1.2, U2.3 (IN2)
Changed lines of the file:
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@@
 		)
 	)
-	(hierarchical_label "IN1"
+	(hierarchical_label "IN2"
 		(shape input)
 		(at 172.72 77.47 0)
@@
 		)
 	)
-	(hierarchical_label "IN2"
+	(hierarchical_label "IN1"
 		(shape input)
 		(at 172.72 82.55 0)
