File: LSPROT2.kicad_sch (KiCad schematic)
At the start: 5 parts, among them U5 VNLD5160TR-E

Commit message: jlc test
Connections:
- net IN1: now also R7.2, U5.3 (IN2); no longer R8.2, U5.1 (IN1)
- net IN2: now also R8.2, U5.1 (IN1); no longer R7.2, U5.3 (IN2)
Changed lines of the file:
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@@
 		)
 	)
-	(hierarchical_label "IN1"
+	(hierarchical_label "IN2"
 		(shape input)
 		(at 187.96 88.9 0)
@@
 		)
 	)
-	(hierarchical_label "IN2"
+	(hierarchical_label "IN1"
 		(shape input)
 		(at 187.96 93.98 0)
